File: Project_Zeta.kicad_pcb (KiCad board)
At the start: 2 copper layers, 80 x 80 mm, 16 parts, among them J1 Conn_01x20, J2 Conn_01x20

Commit message: Init with Rev 1.1
Parts:
- added D3: SS14, Diode_SMD:D_SMA, F.Cu at (159.0, 113.0)
- added D4: SMAJ5.0A, Diode_SMD:D_SMA, F.Cu at (154.0, 115.1)
- added J4: Conn_01x08, Connector_PinHeader_2.54mm:PinHeader_1x08_P2.54mm_Horizontal, F.Cu at (158.6, 87.6)
- added J5: Conn_01x02, Connector_PinHeader_2.54mm:PinHeader_1x02_P2.54mm_Horizontal, F.Cu at (167.8, 110.7)
- added J6: Conn_01x01, Connector_Wire:SolderWire-0.25sqmm_1x01_D0.65mm_OD2mm, F.Cu at (158.5, 127.5)
- added J7: Conn_01x01, Connector_Wire:SolderWire-0.25sqmm_1x01_D0.65mm_OD2mm, F.Cu at (162.5, 127.5)
- added REF**: Fuse_Bourns_MF-RHT050, Fuse:Fuse_Bourns_MF-RHT050, F.Cu at (158.4, 123.0)
- added REF**: CP_Radial_D6.3mm_P2.50mm, Capacitor_THT:CP_Radial_D6.3mm_P2.50mm, F.Cu at (164.5, 117.5)
- added REF**: C_Disc_D5.0mm_W2.5mm_P2.50mm, Capacitor_THT:C_Disc_D5.0mm_W2.5mm_P2.50mm, F.Cu at (169.5, 117.8)
- added RESET1: Conn_01x02_Pin, Connector_PinHeader_2.54mm:PinHeader_1x02_P2.54mm_Vertical, F.Cu at (117.0, 87.3)
- H4: value TerminalBlock_Phoenix_MKDS-1,5-4_1x04_P5.00mm_Horizontal -> TerminalBlock_Phoenix_MKDS-1,5-4_1x04_P5.08mm_Horizontal
- moved H4 0.08 mm to (171.4, 80.0)
Connections:
- H2 pad 3: /GP20 -> /GP18
- H2 pad 4: /GP21 -> /GP19
- J1 pad 9: /GP22 -> unconnected-(J1-GP22-Pad9)
- J2 pad 1: /GP0 -> /GP15
- J2 pad 10: /GP7 -> /GP8
- J2 pad 11: /GP8 -> /GP7
- J2 pad 12: /GP9 -> /GP6
- J2 pad 14: /GP10 -> /GP5
- J2 pad 15: /GP11 -> /GP4
- J2 pad 16: /GP12 -> /GP3
- J2 pad 17: /GP13 -> /GP2
- J2 pad 19: /GP14 -> /GP1
- J2 pad 2: /GP1 -> /GP14
- J2 pad 20: /GP15 -> /GP0
- J2 pad 4: /GP2 -> /GP13
- J2 pad 5: /GP3 -> /GP12
- J2 pad 6: /GP4 -> /GP11
- J2 pad 7: /GP5 -> /GP10
- J2 pad 9: /GP6 -> /GP9
Routing:
- net /3V3_EXT: track 0.00 -> 48.0 mm
- net /GP20: track 74.5 -> 34.4 mm
- net /GP18: track 0.00 -> 39.9 mm
- net /GP21: track 78.9 -> 39.0 mm, vias 2 -> 0
- net /GP19: track 0.00 -> 37.3 mm, vias 0 -> 2
- net GND: track 96.4 -> 127.4 mm, vias 0 -> 1
- net /RUN: track 0.00 -> 19.3 mm
- net /GP8: track 0.00 -> 10.2 mm
- net /GP12: track 0.00 -> 10.2 mm
- net /GP13: track 0.00 -> 10.2 mm
- net /GP11: track 0.00 -> 10.2 mm
- net /GP10: track 0.00 -> 10.2 mm
- net /GP9: track 0.00 -> 10.2 mm
- net /B+: track 0.00 -> 4.49 mm
- net Net-(D3-A): track 0.00 -> 3.20 mm
Other:
- board text added: "*VCC"
- board text added: "3V3_EXT"
- board text added: "B+"
- board text added: "B-"
- board text added: "CSn"
- board text added: "GP8|9"
- board text added: "I2C_0"
- board text added: "Rev 1.1"
- board text added: "SCK"
- board text added: "ϑ"
- board text removed: "Rev 1.0"

Commit message: Updated some nets and added via for some GND point
Connections:
- D3 pad 1: Net-(D3-K) -> /3V3_EXT
- D4 pad 1: Net-(D3-K) -> /3V3_EXT
- D4 pad 2: unconnected-(D4-A2-Pad2) -> GND
- J4 pad 7: /3V3_OUT -> /3V3_EXT
- J6 pad 1: GND -> /B+
Routing:
- net GND: track 127.4 -> 1.00 mm, vias 1 -> 17
- added copper zone on F.Cu, net GND

Commit message: Updated to Rev 1.1
Routing:
- net GND: vias 17 -> 18
Changed lines of the file:
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@@
 	)
 	(gr_text "Design by OatMealXXII"
-		(at 121.75 94.5 0)
+		(at 177.5 101.25 0)
 		(layer "B.SilkS")
 		(effects
@@
 		)
 	)
+	(barcode
+		(at 140.5 118.5 0)
+		(layer "B.SilkS")
+		(size 13 13)
+		(text "https://oatmealxxii.me")
+		(text_height 0.8)
+		(type qr)
+		(ecc_level H)
+		(hide no)
+		(knockout no)
+	)
 	(segment
 		(start 154.035 117.07)
@@
 	)
 	(via
-		(at 108.25 88.25)
+		(at 125.75 100.5)
 		(size 0.6)
 		(drill 0.3)
@@
 	)
 	(via
-		(at 140.25 121.5)
-		(size 0.6)
-		(drill 0.3)
-		(layers "F.Cu" "B.Cu")
-		(free yes)
-		(net "GND")
-	)
-	(via
 		(at 163 123.25)
 		(size 0.6)
@@
 	)
 	(via
-		(at 143.75 111.5)
+		(at 144.25 109.5)
+		(size 0.6)
+		(drill 0.3)
+		(layers "F.Cu" "B.Cu")
+		(free yes)
+		(net "GND")
+	)
+	(via
+		(at 113.5 101.5)
 		(size 0.6)
 		(drill 0.3)
@@
 	(via
 		(at 161.75 115)
+		(size 0.6)
+		(drill 0.3)
+		(layers "F.Cu" "B.Cu")
+		(free yes)
+		(net "GND")
+	)
+	(via
+		(at 114.75 107)
 		(size 0.6)
 		(drill 0.3)
@@
 		(start 121.95 109.95)
 		(end 122.5 110.5)
-		(width 0.2)
+		(width 0.7)
 		(layer "F.Cu")
 		(net "Net-(D1-A)")

Commit message: Updated something IDK I forgotten
Parts:
- C1, C4: renamed from REF**; value CP_Radial_D6.3mm_P2.50mm -> 100uF
- C2, C3: renamed from REF**; value C_Disc_D5.0mm_W2.5mm_P2.50mm -> 0.1uF
- F1, F2: renamed from REF**; value Fuse_Bourns_MF-RHT050 -> Polyfuse
- J3: renamed from Power_in; value TerminalBlock_Phoenix_MKDS-1,5-2_1x02_P5.00mm_Horizontal -> Screw_Terminal_01x02
- moved F2 5.24 mm to (159.6, 118.0), turned to -90 degrees
Connections:
- net 5V renamed +5V
- F2 pad 1: /B+ -> Net-(D3-A)
- F2 pad 2: Net-(D3-A) -> /B+
Changed lines of the file:
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@@
 		(descr "PTC Resettable Fuse, Ihold = 0.5A, Itrip=0.92A, http://www.bourns.com/docs/product-datasheets/mfrht.pdf")
 		(tags "ptc resettable fuse polyfuse THT")
-		(property "Reference" "REF**"
+		(property "Reference" "F1"
 			(at 2.55 -1.9 90)
 			(layer "F.SilkS")
@@
 			)
 		)
-		(property "Value" "Fuse_Bourns_MF-RHT050"
+		(property "Value" "Polyfuse"
 			(at 3.05 -2.4 90)
 			(layer "F.Fab")
@@
 			)
 		)
+		(property ki_fp_filters "*polyfuse* *PTC*")
+		(sheetname "/")
+		(sheetfile "Project_Zeta.kicad_sch")
+		(units
+			(unit
+				(name "A")
+				(pins "1" "2")
+			)
+		)
 		(attr through_hole)
 		(duplicate_pad_numbers_are_jumpers no)
@@
 			(layers "*.Cu" "*.Mask")
 			(remove_unused_layers no)
-			(net "5V")
+			(net "+5V")
+			(pintype "passive")
 		)
 		(pad "2" thru_hole circle
@@
 			(remove_unused_layers no)
 			(net "Net-(D1-A)")
+			(pintype "passive")
 		)
 		(embedded_fonts no)
@@
 	(footprint "Fuse:Fuse_Bourns_MF-RHT050"
 		(layer "F.Cu")
-		(at 158.4 123.05 90)
+		(at 159.6 117.95 -90)
 		(descr "PTC Resettable Fuse, Ihold = 0.5A, Itrip=0.92A, http://www.bourns.com/docs/product-datasheets/mfrht.pdf")
 		(tags "ptc resettable fuse polyfuse THT")
-		(property "Reference" "REF**"
+		(property "Reference" "F2"
 			(at 2.55 -1.9 90)
 			(layer "F.SilkS")
@@
 			)
 		)
-		(property "Value" "Fuse_Bourns_MF-RHT050"
+		(property "Value" "Polyfuse"
 			(at 3.05 -2.4 90)
 			(layer "F.Fab")
@@
 			)
 		)
+		(property ki_fp_filters "*polyfuse* *PTC*")
+		(sheetname "/")
+		(sheetfile "Project_Zeta.kicad_sch")
+		(units
+			(unit
+				(name "A")
+				(pins "1" "2")
+			)
+		)
 		(attr through_hole)
 		(duplicate_pad_numbers_are_jumpers no)
 		(fp_line
-			(start 6.35 -1)
-			(end 6.35 2.2)
+			(start -1.25 2.2)
+			(end -1.25 -1)
 			(stroke
 				(width 0.12)
@@
 		)
 		(fp_line
-			(start 0.578 -1)
-			(end 6.35 -1)
+			(start 4.522 2.2)
+			(end -1.25 2.2)
 			(stroke
 				(width 0.12)
@@
 		)
 		(fp_line
-			(start -1.25 -1)
-			(end -0.578 -1)
+			(start 6.35 2.2)
+			(end 5.678 2.2)
 			(stroke
 				(width 0.12)
@@
 		)
 		(fp_line
-			(start 6.35 2.2)
-			(end 5.678 2.2)
+			(start -1.25 -1)
+			(end -0.578 -1)
 			(stroke
 				(width 0.12)
@@
 		)
 		(fp_line
-			(start 4.522 2.2)
-			(end -1.25 2.2)
+			(start 0.578 -1)
+			(end 6.35 -1)
 			(stroke
 				(width 0.12)
@@
 		)
 		(fp_line
-			(start -1.25 2.2)
-			(end -1.25 -1)
+			(start 6.35 -1)
+			(end 6.35 2.2)
 			(stroke
 				(width 0.12)
@@
 		)
 		(pad "1" thru_hole circle
-			(at 0 0 90)
+			(at 0 0 270)
 			(size 1.71 1.71)
 			(drill 0.71)
 			(layers "*.Cu" "*.Mask")
 			(remove_unused_layers no)
-			(net "/B+")
+			(net "Net-(D3-A)")
+			(pintype "passive")
 		)
 		(pad "2" thru_hole circle
-			(at 5.1 1.2 90)
+			(at 5.1 1.2 270)
 			(size 1.71 1.71)
 			(drill 0.71)
 			(layers "*.Cu" "*.Mask")
 			(remove_unused_layers no)
-			(net "Net-(D3-A)")
+			(net "/B+")
+			(pintype "passive")
 		)
 		(embedded_fonts no)
@@
 		(descr "CP, Radial series, Radial, pin pitch=2.50mm, diameter=6.3mm, height=7mm, Electrolytic Capacitor")
 		(tags "CP Radial series Radial pin pitch 2.50mm diameter 6.3mm height 7mm Electrolytic Capacitor")
-		(property "Reference" "REF**"
+		(property "Reference" "C1"
 			(at -0.317621 -5 0)
 			(layer "F.SilkS")
@@
 			)
 		)
-		(property "Value" "CP_Radial_D6.3mm_P2.50mm"
+		(property "Value" "100uF"
 			(at 0.5 6.5 0)
 			(layer "F.Fab")
@@
 			)
 		)
+		(property ki_fp_filters "CP_*")
+		(sheetname "/")
+		(sheetfile "Project_Zeta.kicad_sch")
+		(units
+			(unit
+				(name "A")
+				(pins "1" "2")
+			)
+		)
 		(attr through_hole)
 		(duplicate_pad_numbers_are_jumpers no)
@@
 			(roundrect_rratio 0.15625)
 			(net "/VSYS")
+			(pintype "passive")
 		)
 		(pad "2" thru_hole circle
@@
 			(remove_unused_layers no)
 			(net "GND")
+			(pintype "passive")
 		)
 		(embedded_fonts no)
@@
 		(descr "CP, Radial series, Radial, pin pitch=2.50mm, diameter=6.3mm, height=7mm, Electrolytic Capacitor")
 		(tags "CP Radial series Radial pin pitch 2.50mm diameter 6.3mm height 7mm Electrolytic Capacitor")
-		(property "Reference" "REF**"
+		(property "Reference" "C4"
 			(at -0.317621 -5 90)
 			(layer "F.SilkS")
@@
 			)
 		)
-		(property "Value" "CP_Radial_D6.3mm_P2.50mm"
+		(property "Value" "100uF"
 			(at 0.5 6.5 90)
 			(layer "F.Fab")
@@
 			)
 		)
+		(property ki_fp_filters "CP_*")
+		(sheetname "/")
+		(sheetfile "Project_Zeta.kicad_sch")
+		(units
+			(unit
+				(name "A")
+				(pins "1" "2")
+			)
+		)
 		(attr through_hole)
 		(duplicate_pad_numbers_are_jumpers no)
@@
 			(roundrect_rratio 0.15625)
 			(net "/3V3_EXT")
+			(pintype "passive")
 		)
 		(pad "2" thru_hole circle
@@
 			(remove_unused_layers no)
 			(net "GND")
+			(pintype "passive")
 		)
 		(embedded_fonts no)
@@
 		(descr "Terminal Block Phoenix MKDS-1,5-2, 2 pins, pitch 5mm, size 10x9.8mm, drill diameter 1.3mm, pad diameter 2.6mm, http://www.farnell.com/datasheets/100425.pdf")
 		(tags "THT Terminal Block Phoenix MKDS-1,5-2 pitch 5mm size 10x9.8mm drill 1.3mm pad 2.6mm")
-		(property "Reference" "Power_in"
+		(property "Reference" "J3"
 			(at -4 -0.1725 90)
 			(layer "F.SilkS")
@@
 			)
 		)
-		(property "Value" "TerminalBlock_Phoenix_MKDS-1,5-2_1x02_P5.00mm_Horizontal"
+		(property "Value" "Screw_Terminal_01x02"
 			(at 1 9.3275 0)
 			(layer "F.Fab")
@@
 			)
 		)
+		(property ki_fp_filters "TerminalBlock*:*")
+		(sheetname "/")
+		(sheetfile "Project_Zeta.kicad_sch")
+		(units
+			(unit
+				(name "A")
+				(pins "1" "2")
+			)
+		)
 		(attr through_hole)
 		(duplicate_pad_numbers_are_jumpers no)
@@
 			(roundrect_rratio 0.096154)
 			(net "GND")
+			(pinfunction "Pin_1_1")
+			(pintype "passive")
 		)
 		(pad "2" thru_hole circle
@@
 			(layers "*.Cu" "*.Mask")
 			(remove_unused_layers no)
-			(net "5V")
+			(net "+5V")
+			(pinfunction "Pin_2_2")
+			(pintype "passive")
 		)
 		(embedded_fonts no)
@@
 		(descr "C, Disc series, Radial, pin pitch=2.50mm, diameter*width=5*2.5mm^2, Capacitor, http://cdn-reichelt.de/documents/datenblatt/B300/DS_KERKO_TC.pdf")
 		(tags "C Disc series Radial pin pitch 2.50mm diameter 5mm width 2.5mm Capacitor")
-		(property "Reference" "REF**"
+		(property "Reference" "C3"
 			(at 1.25 -2.5 90)
 			(layer "F.SilkS")
@@
 			)
 		)
-		(property "Value" "C_Disc_D5.0mm_W2.5mm_P2.50mm"
+		(property "Value" "0.1uF"
 			(at 9 -4.5 0)
 			(layer "F.Fab")
@@
 			)
 		)
+		(property ki_fp_filters "C_*")
+		(sheetname "/")
+		(sheetfile "Project_Zeta.kicad_sch")
+		(units
+			(unit
+				(name "A")
+				(pins "1" "2")
+			)
+		)
 		(attr through_hole)
 		(duplicate_pad_numbers_are_jumpers no)
@@
 			(remove_unused_layers no)
 			(net "/3V3_EXT")
+			(pintype "passive")
 		)
 		(pad "2" thru_hole circle
@@
 			(remove_unused_layers no)
 			(net "GND")
+			(pintype "passive")
 		)
 		(embedded_fonts no)
@@
 		(descr "C, Disc series, Radial, pin pitch=2.50mm, diameter*width=5*2.5mm^2, Capacitor, http://cdn-reichelt.de/documents/datenblatt/B300/DS_KERKO_TC.pdf")
 		(tags "C Disc series Radial pin pitch 2.50mm diameter 5mm width 2.5mm Capacitor")
-		(property "Reference" "REF**"
+		(property "Reference" "C2"
 			(at 1.25 -2.5 0)
 			(layer "F.SilkS")
@@
 			)
 		)
-		(property "Value" "C_Disc_D5.0mm_W2.5mm_P2.50mm"
+		(property "Value" "0.1uF"
 			(at 9 -4.5 90)
 			(layer "F.Fab")
@@
 			)
 		)
+		(property ki_fp_filters "C_*")
+		(sheetname "/")
+		(sheetfile "Project_Zeta.kicad_sch")
+		(units
+			(unit
+				(name "A")
+				(pins "1" "2")
+			)
+		)
 		(attr through_hole)
 		(duplicate_pad_numbers_are_jumpers no)
@@
 			(remove_unused_layers no)
 			(net "/VSYS")
+			(pintype "passive")
 		)
 		(pad "2" thru_hole circle
@@
 			(remove_unused_layers no)
 			(net "GND")
+			(pintype "passive")
 		)
 		(embedded_fonts no)
@@
 	)
 	(via
-		(at 153.75 122.75)
+		(at 155 120)
 		(size 0.6)
 		(drill 0.3)
@@
 	)
 	(segment
-		(start 116.9 120.0725)
-		(end 116.9 115.05)
-		(width 0.7)
-		(layer "F.Cu")
-		(net "5V")
-	)
-	(segment
-		(start 119.5 122.6725)
-		(end 116.9 120.0725)
-		(width 0.7)
-		(layer "F.Cu")
-		(net "5V")
-	)
-	(segment
 		(start 118.1 109.95)
 		(end 120 109.95)
@@
 	)
 	(segment
-		(start 158.5 123.15)
-		(end 158.4 123.05)
+		(start 158.5 127.5)
+		(end 158.5 123.15)
 		(width 0.7)
 		(layer "F.Cu")
@@
 	)
 	(segment
-		(start 158.5 127.5)
-		(end 158.5 123.15)
+		(start 158.5 123.15)
+		(end 158.4 123.05)
 		(width 0.7)
 		(layer "F.Cu")
@@
 		(net "/GP8")
 	)
+	(segment
+		(start 116.9 120.0725)
+		(end 116.9 115.05)
+		(width 0.7)
+		(layer "F.Cu")
+		(net "+5V")
+	)
+	(segment
+		(start 119.5 122.6725)
+		(end 116.9 120.0725)
+		(width 0.7)
+		(layer "F.Cu")
+		(net "+5V")
+	)
 	(zone
